File: hw/lora_devbrd_kicad/devboard.sch (KiCad schematic (older format))
At the start: 32 parts, among them J1 Conn_01x11_Male, J2 Conn_01x11_Male, J3 Conn_01x04_Male, J4 USB_B_Micro, J5 Conn_01x04_Male, J6 Conn_01x04_Male, U1 rhf78-052, U2 LM1117-3.3, U3 FT232RL

Commit message: MISC: [kicad] adds reset button and resistor on SWDIO and SWCLK lines
Parts:
- added R10, R9: 440, Resistor_SMD:R_0805_2012Metric_Pad1.15x1.40mm_HandSolder, symbol Device:R_US
- added SW1: Reset, symbol Switch:SW_Push
- U3: symbol Interface_USB:FT232RL -> devboard-rescue:FT232RL-Interface_USB
Connections:
- wire segments 168 -> 173
Changed lines of the file:
@@
 EESchema Schematic File Version 4
-EELAYER 30 0
+LIBS:devboard-cache
+EELAYER 26 0
 EELAYER END
 $Descr A4 11693 8268
@@
 Text GLabel 1400 2150 2    50   Input ~ 0
 RTS
-Text GLabel 1400 2250 2    50   Input ~ 0
-SWDIO
-Text GLabel 1400 2350 2    50   Input ~ 0
-SWCLK
 Text GLabel 2800 2350 2    50   Input ~ 0
 PA15
@@
 Wire Wire Line
 	1150 2150 1400 2150
-Wire Wire Line
-	1150 2250 1400 2250
-Wire Wire Line
-	1150 2350 1400 2350
 Wire Wire Line
 	2550 1350 2800 1350
@@
 	2650 4800 2650 5050
 $Comp
-L Interface_USB:FT232RL U3
+L devboard-rescue:FT232RL-Interface_USB U3
 U 1 1 5DBDE2AF
 P 8750 2500
@@
 Text Notes 3950 1500 0    50   ~ 0
 What is this ?
+$Comp
+L Device:R_US R9
+U 1 1 5DC1E954
+P 1700 2250
+F 0 "R9" V 1495 2250 50  0000 C CNN
+F 1 "440" V 1600 2250 50  0000 C CNN
+F 2 "Resistor_SMD:R_0805_2012Metric_Pad1.15x1.40mm_HandSolder" V 1740 2240 50  0001 C CNN
+F 3 "~" H 1700 2250 50  0001 C CNN
+	1    1700 2250
+	0    1    1    0
+$EndComp
+$Comp
+L Device:R_US R10
+U 1 1 5DC1E9F0
+P 1700 2350
+F 0 "R10" V 1850 2350 50  0000 C CNN
+F 1 "440" V 1800 2350 50  0000 C CNN
+F 2 "Resistor_SMD:R_0805_2012Metric_Pad1.15x1.40mm_HandSolder" V 1740 2340 50  0001 C CNN
+F 3 "~" H 1700 2350 50  0001 C CNN
+	1    1700 2350
+	0    1    1    0
+$EndComp
+Wire Wire Line
+	1150 2250 1550 2250
+Wire Wire Line
+	1150 2350 1550 2350
+Text GLabel 1950 2250 2    50   Input ~ 0
+SWDIO
+Text GLabel 1950 2350 2    50   Input ~ 0
+SWCLK
+Wire Wire Line
+	1850 2250 1950 2250
+Wire Wire Line
+	1850 2350 1950 2350
+$Comp
+L Switch:SW_Push SW1
+U 1 1 5DC40CA5
+P 5550 4300
+F 0 "SW1" H 5550 4585 50  0000 C CNN
+F 1 "Reset" H 5550 4494 50  0000 C CNN
+F 2 "" H 5550 4500 50  0001 C CNN
+F 3 "" H 5550 4500 50  0001 C CNN
+	1    5550 4300
+	1    0    0    -1
+$EndComp
+$Comp
+L power:GND #PWR019
+U 1 1 5DC41834
+P 5100 4400
+F 0 "#PWR019" H 5100 4150 50  0001 C CNN
+F 1 "GND" H 5105 4227 50  0000 C CNN
+F 2 "" H 5100 4400 50  0001 C CNN
+F 3 "" H 5100 4400 50  0001 C CNN
+	1    5100 4400
+	1    0    0    -1
+$EndComp
+Wire Wire Line
+	5100 4400 5100 4300
+Wire Wire Line
+	5100 4300 5350 4300
+Text GLabel 6000 4300 2    50   Input ~ 0
+nRST
+Wire Wire Line
+	5750 4300 6000 4300
 $EndSCHEMATC

Commit message: MISC: [kicad] sets top layer componetns to it's places
Parts:
- J3: value Conn_01x04_Male -> 3.3V
- J5: value Conn_01x04_Male -> GND
- J6: value Conn_01x04_Male -> LEDS
- J7: renamed from SWD1; value Conn_01x05_Male -> SWD
- SW1: value Reset -> FSM8JSMATR; footprint (none) -> Button_Switch_SMD:SW_SPST_B3S-1000
- renumbered UART1 to J8
Changed lines of the file:
@@
 	9550 1900 9850 1900
 $Comp
-L Connector:Conn_01x02_Male UART1
+L Connector:Conn_01x02_Male J8
 U 1 1 5DC12F97
 P 10050 1900
-F 0 "UART1" H 10022 1782 50  0000 R CNN
+F 0 "J8" H 10022 1782 50  0000 R CNN
 F 1 "Conn_01x02_Male" H 10022 1873 50  0000 R CNN
 F 2 "Connector_PinHeader_2.54mm:PinHeader_1x02_P2.54mm_Vertical" H 10050 1900 50  0001 C CNN
@@
 Connection ~ 1700 7050
 $Comp
-L Connector:Conn_01x05_Male SWD1
+L Connector:Conn_01x05_Male J7
 U 1 1 5DD0C7EC
 P 4400 1900
-F 0 "SWD1" H 4373 1830 50  0000 R CNN
-F 1 "Conn_01x05_Male" H 4373 1921 50  0000 R CNN
+F 0 "J7" H 4373 1830 50  0000 R CNN
+F 1 "SWD" H 4373 1921 50  0000 R CNN
 F 2 "Connector_PinHeader_2.54mm:PinHeader_1x05_P2.54mm_Vertical" H 4400 1900 50  0001 C CNN
 F 3 "~" H 4400 1900 50  0001 C CNN
@@
 P 1150 6250
 F 0 "J3" H 1256 6528 50  0000 C CNN
-F 1 "Conn_01x04_Male" H 1256 6437 50  0000 C CNN
+F 1 "3.3V" H 1256 6437 50  0000 C CNN
 F 2 "Connector_PinHeader_2.54mm:PinHeader_1x04_P2.54mm_Vertical" H 1150 6250 50  0001 C CNN
 F 3 "~" H 1150 6250 50  0001 C CNN
@@
 P 1150 7050
 F 0 "J5" H 1256 7328 50  0000 C CNN
-F 1 "Conn_01x04_Male" H 1256 7237 50  0000 C CNN
+F 1 "GND" H 1256 7237 50  0000 C CNN
 F 2 "Connector_PinHeader_2.54mm:PinHeader_1x04_P2.54mm_Vertical" H 1150 7050 50  0001 C CNN
 F 3 "~" H 1150 7050 50  0001 C CNN
@@
 P 2250 6250
 F 0 "J6" H 2356 6528 50  0000 C CNN
-F 1 "Conn_01x04_Male" H 2356 6437 50  0000 C CNN
+F 1 "LEDS" H 2356 6437 50  0000 C CNN
 F 2 "Connector_PinHeader_2.54mm:PinHeader_1x04_P2.54mm_Vertical" H 2250 6250 50  0001 C CNN
 F 3 "~" H 2250 6250 50  0001 C CNN
@@
 P 5550 4300
 F 0 "SW1" H 5550 4585 50  0000 C CNN
-F 1 "Reset" H 5550 4494 50  0000 C CNN
-F 2 "" H 5550 4500 50  0001 C CNN
+F 1 "FSM8JSMATR" H 5550 4494 50  0000 C CNN
+F 2 "Button_Switch_SMD:SW_SPST_B3S-1000" H 5550 4500 50  0001 C CNN
 F 3 "" H 5550 4500 50  0001 C CNN
 	1    5550 4300
@@
 Wire Wire Line
 	5750 4300 6000 4300
+Connection ~ 4600 3650
 $EndSCHEMATC

Commit message: WIP: [kicad] changed footprints for R and C to 1206
Parts:
- C1, C4, C6: footprint Capacitor_SMD:C_0603_1608Metric_Pad1.05x0.95mm_HandSolder -> Capacitor_SMD:C_1206_3216Metric_Pad1.42x1.75mm_HandSolder
- C2, C3, C5: footprint Capacitor_SMD:C_0805_2012Metric_Pad1.15x1.40mm_HandSolder -> Capacitor_SMD:C_1206_3216Metric_Pad1.42x1.75mm_HandSolder
- R1, R10, R2, R3, R4, R5, R6, R7, R8, R9: footprint Resistor_SMD:R_0805_2012Metric_Pad1.15x1.40mm_HandSolder -> Resistor_SMD:R_1206_3216Metric_Pad1.42x1.75mm_HandSolder
- U3: symbol devboard-rescue:FT232RL-Interface_USB -> Interface_USB:FT232RL
Changed lines of the file:
@@
 EESchema Schematic File Version 4
-LIBS:devboard-cache
-EELAYER 26 0
+EELAYER 30 0
 EELAYER END
 $Descr A4 11693 8268
@@
 F 0 "R1" V 1095 3250 50  0000 C CNN
 F 1 "1K" V 1186 3250 50  0000 C CNN
-F 2 "Resistor_SMD:R_0805_2012Metric_Pad1.15x1.40mm_HandSolder" V 1340 3240 50  0001 C CNN
+F 2 "Resistor_SMD:R_1206_3216Metric_Pad1.42x1.75mm_HandSolder" V 1340 3240 50  0001 C CNN
 F 3 "~" H 1300 3250 50  0001 C CNN
 	1    1300 3250
@@
 F 0 "C1" H 965 4546 50  0000 L CNN
 F 1 "100nF" H 965 4455 50  0000 L CNN
-F 2 "Capacitor_SMD:C_0603_1608Metric_Pad1.05x0.95mm_HandSolder" H 888 4350 50  0001 C CNN
+F 2 "Capacitor_SMD:C_1206_3216Metric_Pad1.42x1.75mm_HandSolder" H 888 4350 50  0001 C CNN
 F 3 "~" H 850 4500 50  0001 C CNN
 	1    850  4500
@@
 	2650 4800 2650 5050
 $Comp
-L devboard-rescue:FT232RL-Interface_USB U3
+L Interface_USB:FT232RL U3
 U 1 1 5DBDE2AF
 P 8750 2500
@@
 F 0 "C4" H 6965 2346 50  0000 L CNN
 F 1 "100nF" H 6965 2255 50  0000 L CNN
-F 2 "Capacitor_SMD:C_0603_1608Metric_Pad1.05x0.95mm_HandSolder" H 6888 2150 50  0001 C CNN
+F 2 "Capacitor_SMD:C_1206_3216Metric_Pad1.42x1.75mm_HandSolder" H 6888 2150 50  0001 C CNN
 F 3 "~" H 6850 2300 50  0001 C CNN
 	1    6850 2300
@@
 F 0 "C5" H 9265 1246 50  0000 L CNN
 F 1 "4.7uF" H 9265 1155 50  0000 L CNN
-F 2 "Capacitor_SMD:C_0805_2012Metric_Pad1.15x1.40mm_HandSolder" H 9188 1050 50  0001 C CNN
+F 2 "Capacitor_SMD:C_1206_3216Metric_Pad1.42x1.75mm_HandSolder" H 9188 1050 50  0001 C CNN
 F 3 "~" H 9150 1200 50  0001 C CNN
 	1    9150 1200
@@
 F 0 "C6" H 9715 1246 50  0000 L CNN
 F 1 "100nF" H 9715 1155 50  0000 L CNN
-F 2 "Capacitor_SMD:C_0603_1608Metric_Pad1.05x0.95mm_HandSolder" H 9638 1050 50  0001 C CNN
+F 2 "Capacitor_SMD:C_1206_3216Metric_Pad1.42x1.75mm_HandSolder" H 9638 1050 50  0001 C CNN
 F 3 "~" H 9600 1200 50  0001 C CNN
 	1    9600 1200
@@
 F 0 "R2" V 5645 6050 50  0000 C CNN
 F 1 "100" V 5736 6050 50  0000 C CNN
-F 2 "Resistor_SMD:R_0805_2012Metric_Pad1.15x1.40mm_HandSolder" V 5890 6040 50  0001 C CNN
+F 2 "Resistor_SMD:R_1206_3216Metric_Pad1.42x1.75mm_HandSolder" V 5890 6040 50  0001 C CNN
 F 3 "~" H 5850 6050 50  0001 C CNN
 	1    5850 6050
@@
 F 0 "R3" V 5645 6400 50  0000 C CNN
 F 1 "100" V 5736 6400 50  0000 C CNN
-F 2 "Resistor_SMD:R_0805_2012Metric_Pad1.15x1.40mm_HandSolder" V 5890 6390 50  0001 C CNN
+F 2 "Resistor_SMD:R_1206_3216Metric_Pad1.42x1.75mm_HandSolder" V 5890 6390 50  0001 C CNN
 F 3 "~" H 5850 6400 50  0001 C CNN
 	1    5850 6400
@@
 F 0 "R4" V 5645 6700 50  0000 C CNN
 F 1 "100" V 5736 6700 50  0000 C CNN
-F 2 "Resistor_SMD:R_0805_2012Metric_Pad1.15x1.40mm_HandSolder" V 5890 6690 50  0001 C CNN
+F 2 "Resistor_SMD:R_1206_3216Metric_Pad1.42x1.75mm_HandSolder" V 5890 6690 50  0001 C CNN
 F 3 "~" H 5850 6700 50  0001 C CNN
 	1    5850 6700
@@
 F 0 "C2" H 9565 5096 50  0000 L CNN
 F 1 "10uF" H 9565 5005 50  0000 L CNN
-F 2 "Capacitor_SMD:C_0805_2012Metric_Pad1.15x1.40mm_HandSolder" H 9488 4900 50  0001 C CNN
+F 2 "Capacitor_SMD:C_1206_3216Metric_Pad1.42x1.75mm_HandSolder" H 9488 4900 50  0001 C CNN
 F 3 "~" H 9450 5050 50  0001 C CNN
 	1    9450 5050
@@
 F 0 "C3" H 10615 5096 50  0000 L CNN
 F 1 "10uF" H 10615 5005 50  0000 L CNN
-F 2 "Capacitor_SMD:C_0805_2012Metric_Pad1.15x1.40mm_HandSolder" H 10538 4900 50  0001 C CNN
+F 2 "Capacitor_SMD:C_1206_3216Metric_Pad1.42x1.75mm_HandSolder" H 10538 4900 50  0001 C CNN
 F 3 "~" H 10500 5050 50  0001 C CNN
 	1    10500 5050
@@
 F 0 "R5" V 3345 6000 50  0000 C CNN
 F 1 "100" V 3436 6000 50  0000 C CNN
-F 2 "Resistor_SMD:R_0805_2012Metric_Pad1.15x1.40mm_HandSolder" V 3590 5990 50  0001 C CNN
+F 2 "Resistor_SMD:R_1206_3216Metric_Pad1.42x1.75mm_HandSolder" V 3590 5990 50  0001 C CNN
 F 3 "~" H 3550 6000 50  0001 C CNN
 	1    3550 6000
@@
 F 0 "R6" V 3345 6200 50  0000 C CNN
 F 1 "100" V 3436 6200 50  0000 C CNN
-F 2 "Resistor_SMD:R_0805_2012Metric_Pad1.15x1.40mm_HandSolder" V 3590 6190 50  0001 C CNN
+F 2 "Resistor_SMD:R_1206_3216Metric_Pad1.42x1.75mm_HandSolder" V 3590 6190 50  0001 C CNN
 F 3 "~" H 3550 6200 50  0001 C CNN
 	1    3550 6200
@@
 F 0 "R7" V 3345 6400 50  0000 C CNN
 F 1 "100" V 3436 6400 50  0000 C CNN
-F 2 "Resistor_SMD:R_0805_2012Metric_Pad1.15x1.40mm_HandSolder" V 3590 6390 50  0001 C CNN
+F 2 "Resistor_SMD:R_1206_3216Metric_Pad1.42x1.75mm_HandSolder" V 3590 6390 50  0001 C CNN
 F 3 "~" H 3550 6400 50  0001 C CNN
 	1    3550 6400
@@
 F 0 "R8" V 3345 6600 50  0000 C CNN
 F 1 "100" V 3436 6600 50  0000 C CNN
-F 2 "Resistor_SMD:R_0805_2012Metric_Pad1.15x1.40mm_HandSolder" V 3590 6590 50  0001 C CNN
+F 2 "Resistor_SMD:R_1206_3216Metric_Pad1.42x1.75mm_HandSolder" V 3590 6590 50  0001 C CNN
 F 3 "~" H 3550 6600 50  0001 C CNN
 	1    3550 6600
@@
 F 0 "R9" V 1495 2250 50  0000 C CNN
 F 1 "440" V 1600 2250 50  0000 C CNN
-F 2 "Resistor_SMD:R_0805_2012Metric_Pad1.15x1.40mm_HandSolder" V 1740 2240 50  0001 C CNN
+F 2 "Resistor_SMD:R_1206_3216Metric_Pad1.42x1.75mm_HandSolder" V 1740 2240 50  0001 C CNN
 F 3 "~" H 1700 2250 50  0001 C CNN
 	1    1700 2250
@@
 F 0 "R10" V 1850 2350 50  0000 C CNN
 F 1 "440" V 1800 2350 50  0000 C CNN
-F 2 "Resistor_SMD:R_0805_2012Metric_Pad1.15x1.40mm_HandSolder" V 1740 2340 50  0001 C CNN
+F 2 "Resistor_SMD:R_1206_3216Metric_Pad1.42x1.75mm_HandSolder" V 1740 2340 50  0001 C CNN
 F 3 "~" H 1700 2350 50  0001 C CNN
 	1    1700 2350

Commit message: WIP: [kicad] Components and designators are placed finally
Other:
- note removed: "C3 must be bigger capacitance, 100?"
- note removed: "Datasheet requires cap be tantalum"
- note removed: "What for?"
- note removed: "What is this ?"
- note removed: "Where D3, R4 are supposed to be located?"
- note removed: "how R and C are chosen?"
Changed lines of the file:
@@
 	1    0    0    -1
 $EndComp
-Text Notes 9350 5200 0    50   ~ 0
-Datasheet requires cap be tantalum
-Text Notes 10300 4950 0    50   ~ 0
-C3 must be bigger capacitance, 100?
-Text Notes 2200 6650 0    50   ~ 0
-What for?
-Text Notes 5000 6900 0    50   ~ 0
-Where D3, R4 are supposed to be located?
-Text Notes 1200 4800 0    50   ~ 0
-how R and C are chosen?
-Text Notes 3950 1500 0    50   ~ 0
-What is this ?
 $Comp
 L Device:R_US R9

Commit message: WIP: [kicad] adds antennas, routing
Parts:
- added J10, J9: Conn_Coaxial_Power, Connector_Coaxial:SMA_Amphenol_132203-12_Horizontal, symbol Connector:Conn_Coaxial_Power
- SW1: footprint Button_Switch_SMD:SW_SPST_B3S-1000 -> Button_Switch_SMD:SW_SPST_EVQPE1
Connections:
- net labels added: ANT_HF, ANT_LF
- wire segments 173 -> 178
- no-connect marks 16 -> 14
Changed lines of the file:
@@
 EESchema Schematic File Version 4
+LIBS:devboard-cache
 EELAYER 30 0
 EELAYER END
@@
 	3550 3650 4600 3650
 Wire Wire Line
-	3550 3250 4600 3250
-Wire Wire Line
-	4600 3250 4600 3450
-Wire Wire Line
 	3550 3450 4600 3450
-Connection ~ 4600 3450
 Wire Wire Line
 	4600 3450 4600 3650
@@
 Wire Wire Line
 	3600 2100 4200 2100
-NoConn ~ 3550 3350
-NoConn ~ 3550 3550
 $Comp
 L power:+5V #PWR0103
@@
 F 0 "SW1" H 5550 4585 50  0000 C CNN
 F 1 "FSM8JSMATR" H 5550 4494 50  0000 C CNN
-F 2 "Button_Switch_SMD:SW_SPST_B3S-1000" H 5550 4500 50  0001 C CNN
-F 3 "" H 5550 4500 50  0001 C CNN
+F 2 "Button_Switch_SMD:SW_SPST_EVQPE1" H 5550 4500 50  0001 C CNN
+F 3 "https://www.chipdip.ru/product/kls7-ts3608-5.0-180-td-02xa" H 5550 4500 50  0001 C CNN
 	1    5550 4300
 	1    0    0    -1
@@
 	5750 4300 6000 4300
 Connection ~ 4600 3650
+Connection ~ 4600 3450
+Wire Wire Line
+	4600 3250 4600 3450
+Wire Wire Line
+	3550 3250 4600 3250
+$Comp
+L Connector:Conn_Coaxial_Power J10
+U 1 1 5DC4C894
+P 5550 2400
+F 0 "J10" V 5775 2350 50  0000 C CNN
+F 1 "Conn_Coaxial_Power" V 5684 2350 50  0000 C CNN
+F 2 "Connector_Coaxial:SMA_Amphenol_132203-12_Horizontal" H 5550 2350 50  0001 C CNN
+F 3 "https://www.chipdip.ru/product/sma-jr50w-br-19-h-73251-220" H 5550 2350 50  0001 C CNN
+	1    5550 2400
+	0    -1   -1   0
+$EndComp
+$Comp
+L Connector:Conn_Coaxial_Power J9
+U 1 1 5DC48EAA
+P 5550 2050
+F 0 "J9" V 5775 2000 50  0000 C CNN
+F 1 "Conn_Coaxial_Power" V 5684 2000 50  0000 C CNN
+F 2 "Connector_Coaxial:SMA_Amphenol_132203-12_Horizontal" H 5550 2000 50  0001 C CNN
+F 3 "https://www.chipdip.ru/product/sma-jr50w-br-19-h-73251-220" H 5550 2000 50  0001 C CNN
+	1    5550 2050
+	0    -1   -1   0
+$EndComp
+Text GLabel 5450 2050 0    50   Input ~ 0
+ANT_LF
+Text GLabel 5450 2400 0    50   Input ~ 0
+ANT_HF
+Text GLabel 3700 3550 2    50   Input ~ 0
+ANT_HF
+Text GLabel 3700 3350 2    50   Input ~ 0
+ANT_LF
+$Comp
+L power:GND #PWR0104
+U 1 1 5DCCAC5F
+P 6050 2400
+F 0 "#PWR0104" H 6050 2150 50  0001 C CNN
+F 1 "GND" H 6055 2227 50  0000 C CNN
+F 2 "" H 6050 2400 50  0001 C CNN
+F 3 "" H 6050 2400 50  0001 C CNN
+	1    6050 2400
+	1    0    0    -1
+$EndComp
+$Comp
+L power:GND #PWR0105
+U 1 1 5DCCB652
+P 6050 2050
+F 0 "#PWR0105" H 6050 1800 50  0001 C CNN
+F 1 "GND" H 6055 1877 50  0000 C CNN
+F 2 "" H 6050 2050 50  0001 C CNN
+F 3 "" H 6050 2050 50  0001 C CNN
+	1    6050 2050
+	1    0    0    -1
+$EndComp
+Wire Wire Line
+	5750 2050 6050 2050
+Wire Wire Line
+	6050 2400 5750 2400
+Wire Wire Line
+	3700 3350 3550 3350
+Wire Wire Line
+	3550 3550 3700 3550
+Wire Wire Line
+	5550 2050 5600 2050
 $EndSCHEMATC
