File: hw/lora_devbrd_kicad/devboard.kicad_pcb (KiCad board)
At the start: 2 copper layers, 64.1 x 58.9 mm, 41 parts, among them J1 Conn_01x11_Male, J10 Conn_Coaxial_Power, J2 Conn_01x11_Male, J3 3.3V, J4 USB_B_Micro, J5 GND, J6 LEDS, J7 SWD, J8 Conn_01x02_Male, J9 Conn_Coaxial_Power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

Commit message: FEAT: [kicad] PCB is ready
Routing:
- net GND: track 137.6 -> 129.2 mm, vias 35 -> 83
- net nRST: track 54.8 -> 55.8 mm
- net SWDIO: track 17.2 -> 17.9 mm
- net +3V3: track 186.7 -> 185.9 mm

Commit message: FEAT: [kicad] removes misplaced via, removes some unneeded gnd routes
Routing:
- net GND: track 129.2 -> 30.3 mm, vias 83 -> 80
- net +3V3: track 185.9 -> 187.3 mm
- net +5V: track 8.28 -> 8.86 mm
Other:
- net class supply added: clearance 0.2, trace_width 0.381, via_dia 0.8, via_drill 0.4
- board text added: "If you can read this you soldered it wrong"

Commit message: MISC: [kicad] add some nice writings ^_^
Other:
- board text added: "2019"
- board text added: "Fox + Urx"
- board text added: "rev 1.0"
Changed lines of the file:
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@@
   (general
     (thickness 1.6)
-    (drawings 43)
+    (drawings 47)
     (tracks 426)
     (zones 0)
@@
     )
   )
+  (gr_text "rev 1.0" (at 121.031 26.416) (layer B.SilkS)
+    (effects (font (size 1.5 1.5) (thickness 0.3)) (justify mirror))
+  )
+  (gr_text 2019 (at 148.082 63.5) (layer B.SilkS)
+    (effects (font (size 1.5 1.5) (thickness 0.3)) (justify mirror))
+  )
+  (gr_line (start 141.986 61.722) (end 154.178 61.722) (layer B.SilkS) (width 0.2))
+  (gr_text "Fox + Urx" (at 148.082 60.198) (layer B.SilkS)
+    (effects (font (size 1.5 1.5) (thickness 0.3)) (justify mirror))
+  )
   (gr_text "If you can read this\nyou soldered it wrong" (at 148.082 46.736) (layer F.SilkS)
